File: Transistor_Calculator_SW_Simulation/Transistor_Calculator_SW_Panel.kicad_sch (KiCad schematic)
At the start: 5 parts, among them Q1 2N3904

Commit message: Other small changes
Parts:
- removed SW1: ~, Button_Switch_THT:Alex_Switch, symbol Switch:SW_Nidec_CAS-120A1
- added D2: LED, LED_THT:LED_D5.0mm_FlatTop, symbol Device:LED
- added R3: 150, Resistor_THT:R_Axial_DIN0204_L3.6mm_D1.6mm_P1.90mm_Vertical, symbol Device:R_US
- added V1, V2: 5, symbol Simulation_SPICE:VDC
Connections:
- net SW1: now reaches R2.2
- net SW1: now also Q1.3 (C), V1.1
- net GND: now reaches R1.1
- net GND: now also R3.2, V1.2, V2.2
- new net: D2.2 (A), V2.1
- new net: D2.1 (K), R3.1
Other:
- moved on the sheet: D1, R1
